File: .out/circuito_generado.kicad_pcb (KiCad board)
At the start: 2 copper layers, 150 x 100 mm, 7 parts, among them U1 DIP-8_W7.62mm

Commit message: Version v1.0.21
Parts:
- moved R2 70.0 mm to (155.0, 30.0)
- moved D1 34.9 mm to (59.0, 82.0)
- moved R1 34.0 mm to (99.0, 30.0)
- moved C2 32.6 mm to (19.0, 82.0)
- moved C1 22.0 mm to (127.0, 30.0)
- moved RV1 14.0 mm to (59.0, 30.0)
- moved U1 6.00 mm to (19.0, 30.0)
Routing:
- net GND: track 105.4 -> 0.00 mm
- net NET_RB_TRIGGER_THRESHOLD: track 86.4 -> 0.00 mm
- net NET_LED_CURRENT_LIMIT: track 48.3 -> 0.00 mm
- net NET_RA_DISCHARGE: track 35.6 -> 0.00 mm
- net NET_LED_OUT: track 28.7 -> 0.00 mm
- net VCC_9V: track 23.1 -> 0.00 mm
- net NET_CONTROL_VOLTAGE: track 15.6 -> 0.00 mm
Other:
- board size 150 x 100 mm -> 170 x 100 mm
